File: documents/PCB/D21_v39.brd (EAGLE design)
At the start: 153.5 x 114 mm, 249 parts, among them SW1 SWT-3, U0 D20BOX, U1 UC3845B, U10 ATSAMD21G1XA-A, U2 LM321MF, U3 TNY254GN, U4 MC34063AD, U5 LM1117MP-3.3, U6 CP2104, U8 ESP-WROOM-32 MODULE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

Commit message: Docs
Parts:
- removed DGND1: (no value), wirepad:4,16O1,6
- removed IO4: (no value), microbuilder_v2:TESTPOINT_ROUND_1MM
- added MI, PAD4, PL: (no value), wirepad:4,16O1,6
- moved DVT3 0.63 mm to (65.2, -36.2)
- moved X3 0.63 mm to (69.2, -29.5)
- moved C32 0.32 mm to (59.4, -24.9)
- moved VD20 0.32 mm to (70.5, -33.7)
- moved RTU 0.16 mm to (46.5, -30.6)
- moved VD25 0.16 mm to (63.5, -30.0)
Connections:
- removed net N$68: IO4.P$1, U8.26
- new net BE: R75.2, U8.30, X5.1
- net BZ: now also U8.26; no longer R75.2, U8.30, X5.1
- net GND: now also PAD4.1; no longer DGND1.1
- net PLUS: now also PL.1
- net SHUNT-: now also MI.1
Routing:
- net BE: track 0.00 -> 145.7 mm, vias 0 -> 4
- net BZ: track 147.0 -> 29.7 mm, vias 5 -> 3
- net N$69: track 55.9 -> 49.8 mm, vias 3 -> 0
- net N$68: track 4.30 -> 0.00 mm
- net +3.3: track 408.5 -> 404.8 mm, vias 13 -> 12
- net KEY: track 185.1 -> 183.7 mm
- net DIN: track 16.4 -> 17.7 mm
- net PGU: track 20.5 -> 19.5 mm, vias 3 -> 1
- net FAN: track 8.14 -> 7.41 mm
- net N$48: track 14.4 -> 15.1 mm
- net N$9: track 7.61 -> 6.97 mm
- net SCL: track 189.1 -> 188.6 mm
- net GND: vias 141 -> 144
Other:
- board text added: "D21.v39"
- board text added: "GND"
- board text added: "LCD 128x128 SPI-3"
- board text added: "LCD 128x160 RGB SPI-3"
- board text added: "R"
- board text added: "SAMD21"
- board text added: "T"
- board text added: "USB"
- board text removed: "D21.v38"
