File: documents/PCB/D21_v39.sch (EAGLE design)
At the start: 249 parts, among them SW1 SWT-3, U0 D20BOX, U1 UC3845B, U10 ATSAMD21G1XA-A, U2 LM321MF, U3 TNY254GN, U4 MC34063AD, U5 LM1117MP-3.3, U6 CP2104, U8 ESP-WROOM-32 MODULE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

Commit message: Docs
Parts:
- removed DGND1: WIREPAD4,16O1,6, wirepad:WIREPAD4,16O1,6
- removed IO4: (no value), microbuilder_v2:TESTPOINTROUND1MM
- added MI, PAD4, PL: WIREPAD4,16O1,6, wirepad:WIREPAD4,16O1,6
Connections:
- removed net N$68: IO4.P$1, U8.IO4
- new net BE: R75.2, U8.IO18, X5.1
- net BZ: now also U8.IO4; no longer R75.2, U8.IO18, X5.1
- net GND: now also PAD4.P; no longer DGND1.P
- net PLUS: now also PL.P
- net SHUNT-: now also MI.P
Other:
- note removed: "(Buzzer or Encoder)"
- moved on the sheet: C15, C17, C20, C21, C25, C26, C27, C28, C37, C38, C39, IO19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
